File: board/pmod-hdmi-tx.sch (KiCad schematic (older format))
At the start: 15 parts, among them P1 PMOD-Device-x2-Type-XHS-Alt, U31 XC9140, U32 REG710-DBV

Commit message: Reorganising the high speed signals.
Connections:
- net HDMI_TX0_CLK+: now also P1.9 (JA4_P); no longer P1.3 (JA2_P)
- net HDMI_TX0_CLK-: now also P1.10 (JA4_N); no longer P1.4 (JA2_N)
- net HDMI_TX0_D0+: now also P1.3 (JA2_P); no longer P1.1 (JA1_P)
- net HDMI_TX0_D0-: now also P1.4 (JA2_N); no longer P1.2 (JA1_N)
- net HDMI_TX0_D1+: now also P1.7 (JA3_P); no longer P1.9 (JA4_P)
- net HDMI_TX0_D1-: now also P1.8 (JA3_N); no longer P1.10 (JA4_N)
- net HDMI_TX0_D2+: now also P1.1 (JA1_P); no longer P1.7 (JA3_P)
- net HDMI_TX0_D2-: now also P1.2 (JA1_N); no longer P1.8 (JA3_N)
Other:
- moved on the sheet: P1
Changed lines of the file:
@@
 Text Label 3300 3000 0    60   ~ 0
 HDMI_TX0_CLK-
+Text Label 1700 3000 2    60   ~ 0
+HDMI_TX0_D0-
 Text Label 3300 2800 0    60   ~ 0
-HDMI_TX0_D0-
-Text Label 1700 3000 2    60   ~ 0
 HDMI_TX0_D1-
 Text Label 1700 2800 2    60   ~ 0
@@
 Text Label 1700 2700 2    60   ~ 0
 HDMI_TX0_D2+
+Text Label 3300 2700 0    60   ~ 0
+HDMI_TX0_D1+
 Text Label 1700 2900 2    60   ~ 0
-HDMI_TX0_D1+
-Text Label 3300 2700 0    60   ~ 0
 HDMI_TX0_D0+
 Text Label 3300 2900 0    60   ~ 0
@@
 F 3 "" H 2500 3450 50  0000 C CNN
 	1    2500 3450
-	-1   0    0    1
+	1    0    0    1
 $EndComp
 Text Label 5150 1125 2    60   ~ 0
@@
 L PMOD-Device-x2-Type-XHS-Alt P1
 U 1 1 58242047
-P 2400 3250
-F 0 "P1" H 2500 3900 60  0000 C CNN
-F 1 "PMOD-Device-x2-Type-XHS-Alt" H 2490 3210 39  0001 C CNN
-F 2 "pmod-conn_6x2:pmod_pin_array_6x2" H 2500 3140 39  0001 C CNN
-F 3 "" H 2500 3550 60  0000 C CNN
-	1    2400 3250
-	1    0    0    -1
-$EndComp
+P 2600 3250
+F 0 "P1" H 2700 3900 60  0000 C CNN
+F 1 "PMOD-Device-x2-Type-XHS-Alt" H 2690 3210 39  0001 C CNN
+F 2 "pmod-conn_6x2:pmod_pin_array_6x2" H 2700 3140 39  0001 C CNN
+F 3 "" H 2700 3550 60  0000 C CNN
+	1    2600 3250
+	-1   0    0    -1
+$EndComp
+Text Notes 1900 4000 0    60   ~ 0
+HDMI High Speed Signals
+Wire Wire Line
+	1700 2700 1825 2700
+Wire Wire Line
+	1825 2700 2100 2700
+Wire Wire Line
+	1700 2800 1875 2800
+Wire Wire Line
+	1875 2800 2100 2800
+Wire Wire Line
+	1700 2900 2025 2900
+Wire Wire Line
+	2025 2900 2100 2900
+Wire Wire Line
+	1700 3000 2075 3000
+Wire Wire Line
+	2075 3000 2100 3000
 Wire Wire Line
 	2900 2700 2925 2700
@@
 	3175 3000 3300 3000
 Wire Wire Line
-	1700 2700 1825 2700
-Wire Wire Line
-	1825 2700 2100 2700
-Wire Wire Line
-	1700 2800 1875 2800
-Wire Wire Line
-	1875 2800 2100 2800
-Wire Wire Line
-	1700 2900 2025 2900
-Wire Wire Line
-	2025 2900 2100 2900
-Wire Wire Line
-	1700 3000 2075 3000
-Wire Wire Line
-	2075 3000 2100 3000
-Wire Wire Line
-	2900 3100 3000 3100
-Wire Wire Line
-	3000 3100 3000 3650
-Wire Wire Line
-	3000 3650 2500 3650
-Wire Wire Line
-	2500 3650 2000 3650
-Wire Wire Line
-	2000 3650 2000 3100
-Wire Wire Line
-	2000 3100 2100 3100
-Wire Wire Line
-	2100 3200 2050 3200
-Wire Wire Line
-	2050 3200 2050 3400
-Wire Wire Line
-	2050 3400 2500 3400
-Wire Wire Line
-	2500 3400 2950 3400
-Wire Wire Line
-	2950 3400 2950 3200
-Wire Wire Line
-	2950 3200 2900 3200
+	2100 3100 2000 3100
+Wire Wire Line
+	2000 3100 2000 3650
+Wire Wire Line
+	2000 3650 2500 3650
+Wire Wire Line
+	2500 3650 3000 3650
+Wire Wire Line
+	3000 3650 3000 3100
+Wire Wire Line
+	3000 3100 2900 3100
+Wire Wire Line
+	2900 3200 2950 3200
+Wire Wire Line
+	2950 3200 2950 3400
+Wire Wire Line
+	2950 3400 2500 3400
+Wire Wire Line
+	2500 3400 2050 3400
+Wire Wire Line
+	2050 3400 2050 3200
+Wire Wire Line
+	2050 3200 2100 3200
 Wire Wire Line
 	2500 3700 2500 3650
@@
 Wire Wire Line
 	3125 2250 4150 2250
+Connection ~ 3175 3000
+Wire Wire Line
+	2025 2000 4150 2000
+Connection ~ 3125 2900
+Wire Wire Line
+	2925 1750 4150 1750
+Connection ~ 2975 2800
+Wire Wire Line
+	1825 1500 4150 1500
+Connection ~ 2925 2700
+Wire Wire Line
+	1875 1600 4150 1600
+Wire Wire Line
+	2975 1850 4150 1850
+Connection ~ 1875 2800
+Wire Wire Line
+	2075 2100 4150 2100
+Connection ~ 2025 2900
+Wire Wire Line
+	3175 2350 4150 2350
 Connection ~ 2075 3000
-Wire Wire Line
-	2925 2000 4150 2000
-Connection ~ 2025 2900
-Wire Wire Line
-	2025 1750 4150 1750
-Connection ~ 1875 2800
-Wire Wire Line
-	1825 2700 1825 1500
-Wire Wire Line
-	1825 1500 4150 1500
-Connection ~ 1825 2700
-Wire Wire Line
-	1875 1600 4150 1600
-Wire Wire Line
-	2075 1850 4150 1850
-Connection ~ 2975 2800
-Wire Wire Line
-	2975 2100 4150 2100
-Connection ~ 3125 2900
-Wire Wire Line
-	3175 2350 4150 2350
-Connection ~ 3175 3000
 Wire Wire Line
 	6250 2000 7275 2000
@@
 Wire Wire Line
 	4700 1125 4700 1100
-Wire Wire Line
-	1875 2800 1875 1600
-Wire Wire Line
-	2025 2900 2025 1750
-Wire Wire Line
-	2075 3000 2075 1850
-Wire Wire Line
-	2925 2700 2925 2000
-Connection ~ 2925 2700
-Wire Wire Line
-	2975 2100 2975 2800
+Connection ~ 1825 2700
 Wire Wire Line
 	3125 2900 3125 2250
 Wire Wire Line
-	3175 3000 3175 2350
-Text Notes 1900 4000 0    60   ~ 0
-HDMI High Speed Signals
+	3175 2350 3175 3000
+Wire Wire Line
+	2025 2900 2025 2000
+Wire Wire Line
+	2075 2100 2075 3000
+Wire Wire Line
+	2925 2700 2925 1750
+Wire Wire Line
+	2975 1850 2975 2800
+Wire Wire Line
+	1825 2700 1825 1500
+Wire Wire Line
+	1875 1600 1875 2800
 $EndSCHEMATC

Commit message: Reworking stuff.
Changed lines of the file:
@@
 HDMI High Speed Signals
 Wire Wire Line
-	1700 2700 1825 2700
-Wire Wire Line
-	1825 2700 2100 2700
-Wire Wire Line
-	1700 2800 1875 2800
-Wire Wire Line
-	1875 2800 2100 2800
-Wire Wire Line
-	1700 2900 2025 2900
-Wire Wire Line
-	2025 2900 2100 2900
-Wire Wire Line
-	1700 3000 2075 3000
-Wire Wire Line
-	2075 3000 2100 3000
-Wire Wire Line
-	2900 2700 2925 2700
-Wire Wire Line
-	2925 2700 3300 2700
-Wire Wire Line
-	2900 2800 2975 2800
-Wire Wire Line
-	2975 2800 3300 2800
-Wire Wire Line
-	2900 2900 3125 2900
-Wire Wire Line
-	3125 2900 3300 2900
-Wire Wire Line
-	2900 3000 3175 3000
-Wire Wire Line
-	3175 3000 3300 3000
+	1700 2700 2100 2700
+Wire Wire Line
+	1700 2800 2100 2800
+Wire Wire Line
+	1700 2900 2100 2900
+Wire Wire Line
+	1700 3000 2100 3000
+Wire Wire Line
+	2900 2700 3300 2700
+Wire Wire Line
+	2900 2800 3300 2800
+Wire Wire Line
+	2900 2900 3300 2900
+Wire Wire Line
+	2900 3000 3300 3000
 Wire Wire Line
 	2100 3100 2000 3100
@@
 	2000 3100 2000 3650
 Wire Wire Line
-	2000 3650 2500 3650
-Wire Wire Line
-	2500 3650 3000 3650
+	2000 3650 3000 3650
 Wire Wire Line
 	3000 3650 3000 3100
@@
 	2900 3200 2950 3200
 Wire Wire Line
-	2950 3200 2950 3400
-Wire Wire Line
-	2950 3400 2500 3400
-Wire Wire Line
-	2500 3400 2050 3400
+	2950 3400 2950 3200
+Wire Wire Line
+	2050 3400 2950 3400
 Wire Wire Line
 	2050 3400 2050 3200
@@
 	6250 2000 7275 2000
 Wire Wire Line
-	6250 2100 7650 2100
-Wire Wire Line
-	7650 2100 7700 2100
-Wire Wire Line
-	6250 2250 6875 2250
-Wire Wire Line
-	6875 2250 7975 2250
-Wire Wire Line
-	6250 2350 6875 2350
-Wire Wire Line
-	6875 2350 7975 2350
-Wire Wire Line
-	6250 2500 6775 2500
-Wire Wire Line
-	6775 2500 7975 2500
-Wire Wire Line
-	6250 2600 6925 2600
-Wire Wire Line
-	6925 2600 7975 2600
+	6250 2100 7700 2100
+Wire Wire Line
+	6250 2250 7975 2250
+Wire Wire Line
+	6250 2350 7975 2350
+Wire Wire Line
+	6250 2500 7975 2500
+Wire Wire Line
+	6250 2600 7975 2600
 Wire Wire Line
 	4700 1125 5250 1125
@@
 	1900 6675 1500 6675
 Wire Wire Line
-	800  6825 950  6825
-Wire Wire Line
-	950  6825 1900 6825
-Wire Wire Line
-	950  6525 950  6675
-Wire Wire Line
-	950  6675 950  6825
-Wire Wire Line
-	950  6825 950  6925
+	800  6825 1900 6825
+Wire Wire Line
+	950  6525 950  6925
 Wire Wire Line
 	950  6525 1050 6525
@@
 Connection ~ 950  6825
 Wire Wire Line
-	3000 6575 3550 6575
-Wire Wire Line
-	3550 6575 4175 6575
+	3000 6575 4175 6575
 Connection ~ 3550 6575
 Wire Wire Line
@@
 	3050 6775 3050 7275
 Wire Wire Line
-	3550 6925 3550 7275
-Wire Wire Line
-	3550 7275 3550 7400
+	3550 6925 3550 7400
 Wire Notes Line
 	650  6275 3200 6275
@@
 	950  7225 950  7275
 Wire Wire Line
-	950  7275 3050 7275
-Wire Wire Line
-	3050 7275 3550 7275
-Wire Wire Line
-	3550 7275 5250 7275
-Wire Wire Line
-	5250 7275 6050 7275
+	950  7275 6050 7275
 Wire Wire Line
 	6250 1500 8125 1500
@@
 	7575 2000 7650 2000
 Wire Wire Line
-	7650 2000 7650 2100
-Wire Wire Line
-	7650 2100 7650 2175
+	7650 2000 7650 2175
 Connection ~ 7650 2100
 Wire Wire Line
@@
 	6775 2975 6775 3175
 Wire Wire Line
-	6775 3175 6850 3175
-Wire Wire Line
-	6850 3175 6925 3175
+	6775 3175 6925 3175
 Wire Wire Line
 	6925 3175 6925 2975
@@
 Connection ~ 6850 3175
 Wire Wire Line
-	6325 6775 6050 6775
-Wire Wire Line
-	6050 6775 5800 6775
-Wire Wire Line
-	6325 6500 6325 6575
-Wire Wire Line
-	6325 6575 6325 6775
+	6325 6775 5800 6775
+Wire Wire Line
+	6325 6500 6325 6775
 Wire Wire Line
 	4625 6525 4700 6525
@@
 	3950 7450 3950 6275
 Wire Wire Line
-	3550 6000 3550 6575
-Wire Wire Line
-	3550 6575 3550 6625
+	3550 6000 3550 6625
 Wire Wire Line
 	6225 6575 6325 6575
