File: board/pmod-hdmi-rx.sch (KiCad schematic (older format))
At the start: 20 parts, among them P1 PMOD-CONN_6X2, U31 XC9140, U32 REG710-DBV

Commit message: Update from templates + s/HPD/HOT/ + s/HPA/HOT/
Other:
- note added: "On PRX0\n - SCL on Pin X\n - SDA on Pin X\n - CEC on Pin X\n - HOT on Pin X"
- note removed: "On PRX0\n - SCL on Pin X\n - SDA on Pin X\n - CEC on Pin X\n - HPD on Pin X"
Changed lines of the file:
@@
 F13 "HDMI_RX0_TXEN" I R 6250 2250 60
 F14 "HDMI_RX0_PEEN" I R 6250 2350 60
-F15 "HDMI_RX0_HPA" I R 6250 1800 60
+F15 "HDMI_RX0_HOT" I R 6250 1800 60
 F16 "HDMI_RX0_IO0" B R 6250 2500 60
 F17 "HDMI_RX0_IO1" B R 6250 2600 60
@@
 HDMI_RX0_CEC
 Text Label 8125 1800 0    60   ~ 0
-HDMI_RX0_HPD
+HDMI_RX0_HOT
 Text Notes 8875 1850 0    60   ~ 0
-On PRX0\n - SCL on Pin X\n - SDA on Pin X\n - CEC on Pin X\n - HPD on Pin X
+On PRX0\n - SCL on Pin X\n - SDA on Pin X\n - CEC on Pin X\n - HOT on Pin X
 Text Notes 1850 4200 0    60   ~ 0
 HDMI High Speed Signals\nPositive signals on Top Row\nNegative signals on Bottom Row

Commit message: Adding CE for XC9140 part.
Connections:
- net HDMI_RX0_IO0: now also R31.1, U31.1 (CE)
Changed lines of the file:
@@
 Text Notes 7100 4425 0    79   ~ 16
 EDID EEPROM
+Wire Wire Line
+	1750 6675 1750 6050
+Wire Wire Line
+	1750 6050 1900 6050
+Connection ~ 1750 6675
+Text Label 1900 6050 0    60   ~ 0
+HDMI_RX0_IO0
 $EndSCHEMATC
