File: board/hdmi_RX0.sch (KiCad schematic (older format))
At the start: 21 parts

Commit message: Updating from template.
Parts:
- removed CTX001, CTX002, CTX003, CTX004, CTX005, CTX006, CTX007, CTX008: 0.1uF, Capacitors_SMD:C_0402, symbol C_Small
- removed CTX013: 10n, Capacitors_SMD:C_0402, symbol C_Small
- removed CTX016, CTX017: 0.1uF, Capacitors_SMD:C_0402, symbol C
- removed DTX001: D, Diodes_SMD:SOD-523, symbol D
- removed JTX0: HDMI_OUT, hdmi:HDMI_TH, symbol HDMI_OUT
- removed PTX0: PMOD-CONN_6X2, pmod:pmod_pin_array_6x2, symbol PMOD-CONN_6X2
- removed RTX001, RTX002, RTX004, RTX005: 2k2, Resistors_SMD:R_0402, symbol R
- removed RTX003: 12k4, Resistors_SMD:R_0402, symbol R
- removed RTX008: 27K, Resistors_SMD:R_0402, symbol R
- removed UTX0: PTN3363, Housings_DFN_QFN:QFN-32-1EP_5x5mm_Pitch0.5mm, symbol PTN3363
- added CRX001, CRX002, CRX003: 10uF, Capacitors_SMD:C_0603, symbol C
- added CRX004, CRX005, CRX006, CRX007, CRX010: 0.1uF, Capacitors_SMD:C_0402, symbol C
- added CRX008, CRX009, CRX011, CRX012, CRX014: 10nF, Capacitors_SMD:C_0402, symbol C
- added CRX013: 0.1nF, Capacitors_SMD:C_0402, symbol C
- added CRX015: 10uF, Capacitors_SMD:C_0402, symbol C
- added DRX001: LED, LEDs:LED_0603, symbol LED
- added DRX002, DRX003: D, Diodes_SMD:SOD-123, symbol D
- added FBRX001, FBRX002, FBRX003, FBRX004: FILTER, Capacitors_SMD:C_0805, symbol FILTER
- added JRX0: HDMI_IN, hdmi:HDMI_TH, symbol HDMI_IN
- added PRX0: PMOD-CONN_6X2, pmod:pmod_pin_array_6x2, symbol PMOD-CONN_6X2
- added QRX001, QRX002, QRX003: FDV301N, TO_SOT_Packages_SMD:SOT-23, symbol FDV301N
- added RRX001, RRX002, RRX006, RRX007, RRX008: 100K, Resistors_SMD:R_0402, symbol R
- added RRX003, RRX010, RRX012: 1K, Resistors_SMD:R_0402, symbol R
- added RRX004: 560R, Resistors_SMD:R_0402, symbol R
- added RRX005: 2K, Resistors_SMD:R_0402, symbol R
- added RRX009, RRX011: 47K, Resistors_SMD:R_0402, symbol R
- added URX0: AD8195, Housings_DFN_QFN:QFN-40-1EP_6x6mm_Pitch0.5mm, symbol AD8195
Connections:
- net GND: now also CRX001.2, CRX002.2, CRX003.2, CRX004.2, CRX005.2, CRX006.2, CRX007.2, CRX008.2, CRX009.2, CRX010.2, CRX011.2, CRX012.2, CRX013.2, CRX014.2, CRX015.2, JRX0.17 (DDC/CEC/HEC), JRX0.2 (D2S), JRX0.5 (D1S), JRX0.8 (D0S), PRX0.11 (P11), PRX0.5 (P5), QRX001.2, QRX002.2, QRX003.2, RRX001.1, RRX007.2, RRX008.2, URX0.24 (AVEE), URX0.27 (AVEE), URX0.37 (AVEE), URX0.41 (AVEE)
- net VCC3V3: now also FBRX001.1, FBRX002.1, FBRX003.1, PRX0.12 (P12), PRX0.6 (P6), RRX006.1, RRX010.2, RRX012.2, URX0.33 (VREF-OUT)
- new net: CRX015.1, URX0.21 (COMP)
- new net: CRX013.1, CRX014.1, DRX002.1 (K), DRX003.1 (K), URX0.32 (AMUX), URX0.36 (VREF-IN)
- new net: JRX0.11 (CLKS), RRX005.2
- new net: FBRX004.1, JRX0.18 (+5V)
- new net: QRX001.3, QRX002.1, RRX002.1
- new net: QRX003.3, RRX004.1
- new net: DRX001.1 (K), RRX004.2
- new net AVCC3V3: CRX001.1, CRX004.1, CRX007.1, CRX010.1, CRX011.1, CRX012.1, FBRX001.2, URX0.10 (AVCC), URX0.16 (AVCC), URX0.22 (AVCC), URX0.23 (AVCC), URX0.25 (AVCC), URX0.26 (AVCC), URX0.30 (AVCC)
- new net HDMIP_RX0_CEC: JRX0.13 (CEC), URX0.38 (CEC-IN)
- new net HDMIP_RX0_CLK+: JRX0.10 (CLK+), URX0.2 (IP0)
- new net HDMIP_RX0_CLK-: JRX0.12 (CLK-), RRX005.1, URX0.1 (IN0)
- new net HDMIP_RX0_D0+: JRX0.7 (D0+), URX0.4 (IP1)
- new net HDMIP_RX0_D0-: JRX0.9 (D0-), URX0.3 (IN1)
- new net HDMIP_RX0_D1+: JRX0.4 (D1+), URX0.7 (IP2)
- new net HDMIP_RX0_D1-: JRX0.6 (D1-), URX0.6 (IN2)
- new net HDMIP_RX0_D2+: JRX0.1 (D2+), URX0.9 (IP3)
- new net HDMIP_RX0_D2-: JRX0.3 (D2-), URX0.8 (IN3)
- new net HDMIP_RX0_HPD: JRX0.19 (HPD), QRX002.3, QRX003.1, RRX003.1
- new net HDMIP_RX0_SCL: JRX0.15 (SCL), RRX009.1, URX0.40 (SCL-IN)
- new net HDMIP_RX0_SDA: JRX0.16 (SDA), RRX011.1, URX0.39 (SDA-IN)
- new net HDMI_RX0_CEC: PRX0.1 (P1), URX0.31 (CEC-OUT)
- new net HDMI_RX0_CLK+: URX0.12 (OP0)
- new net HDMI_RX0_CLK-: URX0.11 (ON0)
- new net HDMI_RX0_D0+: URX0.15 (OP1)
- new net HDMI_RX0_D0-: URX0.14 (ON1)
- new net HDMI_RX0_D1+: URX0.18 (OP2)
- new net HDMI_RX0_D1-: URX0.17 (ON2)
- new net HDMI_RX0_D2+: URX0.20 (OP3)
- new net HDMI_RX0_D2-: URX0.19 (ON3)
- new net HDMI_RX0_HPA: PRX0.4 (P4), QRX001.1, RRX001.2
- new net HDMI_RX0_IO0: PRX0.7 (P7)
- new net HDMI_RX0_IO1: PRX0.8 (P8)
- new net HDMI_RX0_PEEN: PRX0.10 (P10), RRX006.2, RRX007.1, URX0.29 (PE-EN)
- new net HDMI_RX0_SCL: PRX0.2 (P2), RRX010.1, URX0.35 (SCL-OUT)
- new net HDMI_RX0_SDA: PRX0.3 (P3), RRX012.1, URX0.34 (SDA-OUT)
- new net HDMI_RX0_TXEN: PRX0.9 (P9), RRX008.1, URX0.28 (TX-EN)
- new net VCC5V0: DRX002.2 (A)
- new net VCC5V0_RX0: DRX001.2 (A), DRX003.2 (A), FBRX004.2, RRX002.2, RRX003.2, RRX009.2, RRX011.2
- new net VTTI3V3: CRX003.1, CRX006.1, CRX009.1, FBRX003.2, URX0.5 (VTTI)
- new net VTTO3V3: CRX002.1, CRX005.1, CRX008.1, FBRX002.2, URX0.13 (VTTO)

Commit message: Update from template.
Connections:
- net HDMI_RX0_CEC: now also PRX0.7 (P7); no longer PRX0.1 (P1)
- net HDMI_RX0_HPA: now also PRX0.2 (P2); no longer PRX0.4 (P4), QRX001.1, RRX001.2
- net HDMI_RX0_IO0: now also PRX0.9 (P9); no longer PRX0.7 (P7)
- net HDMI_RX0_IO1: now also PRX0.3 (P3); no longer PRX0.8 (P8)
- net HDMI_RX0_PEEN: now also PRX0.4 (P4); no longer PRX0.10 (P10)
- net HDMI_RX0_SCL: now also PRX0.1 (P1); no longer PRX0.2 (P2)
- net HDMI_RX0_SDA: now also PRX0.8 (P8); no longer PRX0.3 (P3)
- net HDMI_RX0_TXEN: now also PRX0.10 (P10); no longer PRX0.9 (P9)
- new net HDMI_RX0_HPD: QRX001.1, RRX001.2
Other:
- note added: "Do not populate"
- note added: "This sheet is generated from ../external/templates/\nDO NOT MODIFY!!!\ne23ffb6"
- note removed: "This sheet is generated from ../external/templates/\nDO NOT MODIFY!!!\n1620b96"
Changed lines of the file:
@@
 LIBS:contrib
 LIBS:valves
-LIBS:pmod
+LIBS:pmod-conn_6x2
+LIBS:ma78l00
+LIBS:fdv301n
 LIBS:hdmi
-LIBS:ma78l00
-LIBS:pmod-conn_6x2
-LIBS:EEPROM
-LIBS:xc9140
-LIBS:reg710-dbv
 LIBS:ad8195
-LIBS:fdv301n
-LIBS:pmod-hdmi-rx-cache
 EELAYER 25 0
 EELAYER END
 $Descr A3 16535 11693
 encoding utf-8
-Sheet 2 2
+Sheet 1 1
 Title ""
 Date ""
@@
 Text HLabel 10100 3500 2    60   BiDi ~ 0
 HDMI_RX0_SDA
-Text HLabel 6050 4900 0    60   Input ~ 0
+Text HLabel 5770 4900 0    60   Input ~ 0
 HDMI_RX0_TXEN
-Text HLabel 6050 5000 0    60   Input ~ 0
+Text HLabel 5770 5000 0    60   Input ~ 0
 HDMI_RX0_PEEN
+Text Label 7560 6600 2    60   ~ 0
+HDMI_RX0_SCL
 Text Label 4820 6700 0    60   ~ 0
-HDMI_RX0_SCL
-Text Label 4820 6800 0    60   ~ 0
 HDMI_RX0_SDA
 Text Label 5170 7100 0    60   ~ 0
@@
 Text Label 6150 4000 2    60   ~ 0
 HDMIP_RX0_HPD
-Text Label 3100 6050 0    60   ~ 0
+Text Label 3525 5785 1    60   ~ 0
 HDMIP_RX0_HPD
 Text Label 1500 6600 0    60   ~ 0
-HDMI_RX0_HPA
+HDMI_RX0_HPD
 Text Label 1500 7150 0    60   ~ 0
 GND
-Text Label 4820 6900 0    60   ~ 0
+Text Label 7560 6700 2    60   ~ 0
 HDMI_RX0_HPA
 Text Label 6750 1750 0    60   ~ 0
 GND
 Text HLabel 1500 6600 0    60   Input ~ 0
-HDMI_RX0_HPA
+HDMI_RX0_HPD
 Text Notes 615  11035 0    197  ~ 39
-This sheet is generated from ../external/templates/\nDO NOT MODIFY!!!\n1620b96
+This sheet is generated from ../external/templates/\nDO NOT MODIFY!!!\ne23ffb6
 Text Label 4820 6600 0    60   ~ 0
 HDMI_RX0_CEC
-Text Label 7560 6700 2    60   ~ 0
+Text Label 7560 6800 2    60   ~ 0
 HDMI_RX0_IO1
-Text Label 7560 6800 2    60   ~ 0
+Text Label 4820 6900 0    60   ~ 0
 HDMI_RX0_TXEN
 Text Label 7560 6900 2    60   ~ 0
 HDMI_RX0_PEEN
-Text Label 7560 6600 2    60   ~ 0
+Text Label 4820 6800 0    60   ~ 0
 HDMI_RX0_IO0
-Text HLabel 7560 6600 2    60   BiDi ~ 0
+Text HLabel 4820 6800 0    60   BiDi ~ 0
 HDMI_RX0_IO0
-Text HLabel 7560 6700 2    60   BiDi ~ 0
+Text HLabel 7560 6800 2    60   BiDi ~ 0
 HDMI_RX0_IO1
 Text HLabel 10100 2100 2    60   Output ~ 0
@@
 	7150 3650 6950 3650
 Wire Wire Line
-	6950 3650 6950 4900
-Wire Wire Line
-	6950 4900 6050 4900
+	6950 4900 6950 3650
+Wire Wire Line
+	5770 4900 6950 4900
 Wire Wire Line
 	7150 3750 7050 3750
 Wire Wire Line
-	7050 3750 7050 5000
-Wire Wire Line
-	7050 5000 6050 5000
+	7050 5000 7050 3750
+Wire Wire Line
+	5770 5000 7050 5000
 Wire Wire Line
 	6600 4900 6600 5150
@@
 F 3 "" H 6150 6850 60  0000 C CNN
 	1    6150 6850
-	1    0    0    -1
-$EndComp
+	-1   0    0    -1
+$EndComp
+Wire Notes Line
+	5965 4135 5965 5735
+Wire Notes Line
+	5965 5735 6805 5735
+Wire Notes Line
+	6805 5735 6805 4135
+Wire Notes Line
+	6805 4135 5965 4135
+Text Notes 5995 4240 0    60   ~ 0
+Do not populate
+Wire Wire Line
+	3525 5785 3525 6050
+Connection ~ 3525 6050
 $EndSCHEMATC

Commit message: Adding footprints.
Parts:
- CRX015: footprint Capacitors_SMD:C_0402 -> Capacitors_SMD:C_0603
Changed lines of the file:
@@
 LIBS:contrib
 LIBS:valves
+LIBS:pmod
+LIBS:hdmi
+LIBS:ma78l00
 LIBS:pmod-conn_6x2
-LIBS:ma78l00
+LIBS:EEPROM
+LIBS:xc9140
+LIBS:reg710-dbv
+LIBS:ad8195
 LIBS:fdv301n
-LIBS:hdmi
-LIBS:ad8195
+LIBS:pmod-hdmi-rx-cache
 EELAYER 25 0
 EELAYER END
 $Descr A3 16535 11693
 encoding utf-8
-Sheet 1 1
+Sheet 2 2
 Title ""
 Date ""
@@
 $EndComp
 $Comp
-L GND #PWR102
+L GND #PWR014
 U 1 1 57C0819F
 P 7850 4300
-F 0 "#PWR102" H 7850 4050 60  0001 C CNN
+F 0 "#PWR014" H 7850 4050 60  0001 C CNN
 F 1 "GND" H 7850 4150 60  0000 C CNN
 F 2 "" H 7850 4300 60  0000 C CNN
@@
 F 0 "CRX015" H 9100 4100 50  0000 L CNN
 F 1 "10uF" H 9100 3900 50  0000 L CNN
-F 2 "Capacitors_SMD:C_0402" H 9088 3850 30  0001 C CNN
+F 2 "Capacitors_SMD:C_0603" H 9088 3850 30  0001 C CNN
 F 3 "" H 9050 4000 60  0000 C CNN
 	1    9050 4000
@@
 $EndComp
 $Comp
-L GND #PWR101
+L GND #PWR015
 U 1 1 57C093D2
 P 6850 1800
-F 0 "#PWR101" H 6850 1550 60  0001 C CNN
+F 0 "#PWR015" H 6850 1550 60  0001 C CNN
 F 1 "GND" H 6850 1650 60  0000 C CNN
 F 2 "" H 6850 1800 60  0000 C CNN
@@
 	7150 3650 6950 3650
 Wire Wire Line
-	6950 4900 6950 3650
-Wire Wire Line
-	5770 4900 6950 4900
+	6950 3650 6950 4900
+Wire Wire Line
+	6950 4900 5770 4900
 Wire Wire Line
 	7150 3750 7050 3750
 Wire Wire Line
-	7050 5000 7050 3750
-Wire Wire Line
-	5770 5000 7050 5000
+	7050 3750 7050 5000
+Wire Wire Line
+	7050 5000 5770 5000
 Wire Wire Line
 	6600 4900 6600 5150

Commit message: Updating from template.
Other:
- note added: "This sheet is generated from ../external/templates/\nDO NOT MODIFY!!!\nedd182c"
- note removed: "This sheet is generated from ../external/templates/\nDO NOT MODIFY!!!\ne23ffb6"
Changed lines of the file:
@@
 LIBS:contrib
 LIBS:valves
-LIBS:pmod
+LIBS:pmod-conn_6x2
+LIBS:ma78l00
+LIBS:fdv301n
 LIBS:hdmi
-LIBS:ma78l00
-LIBS:pmod-conn_6x2
-LIBS:EEPROM
-LIBS:xc9140
-LIBS:reg710-dbv
 LIBS:ad8195
-LIBS:fdv301n
-LIBS:pmod-hdmi-rx-cache
 EELAYER 25 0
 EELAYER END
 $Descr A3 16535 11693
 encoding utf-8
-Sheet 2 2
+Sheet 1 1
 Title ""
 Date ""
@@
 $EndComp
 $Comp
-L GND #PWR014
+L GND #PWR102
 U 1 1 57C0819F
 P 7850 4300
-F 0 "#PWR014" H 7850 4050 60  0001 C CNN
+F 0 "#PWR102" H 7850 4050 60  0001 C CNN
 F 1 "GND" H 7850 4150 60  0000 C CNN
 F 2 "" H 7850 4300 60  0000 C CNN
@@
 $EndComp
 $Comp
-L GND #PWR015
+L GND #PWR101
 U 1 1 57C093D2
 P 6850 1800
-F 0 "#PWR015" H 6850 1550 60  0001 C CNN
+F 0 "#PWR101" H 6850 1550 60  0001 C CNN
 F 1 "GND" H 6850 1650 60  0000 C CNN
 F 2 "" H 6850 1800 60  0000 C CNN
@@
 HDMI_RX0_HPD
 Text Notes 615  11035 0    197  ~ 39
-This sheet is generated from ../external/templates/\nDO NOT MODIFY!!!\ne23ffb6
+This sheet is generated from ../external/templates/\nDO NOT MODIFY!!!\nedd182c
 Text Label 4820 6600 0    60   ~ 0
 HDMI_RX0_CEC
@@
 	7150 3650 6950 3650
 Wire Wire Line
-	6950 3650 6950 4900
-Wire Wire Line
-	6950 4900 5770 4900
+	6950 4900 6950 3650
+Wire Wire Line
+	5770 4900 6950 4900
 Wire Wire Line
 	7150 3750 7050 3750
 Wire Wire Line
-	7050 3750 7050 5000
-Wire Wire Line
-	7050 5000 5770 5000
+	7050 5000 7050 3750
+Wire Wire Line
+	5770 5000 7050 5000
 Wire Wire Line
 	6600 4900 6600 5150

Commit message: Update from templates + s/HPD/HOT/ + s/HPA/HOT/
Connections:
- net HDMI_RX0_HPD is gone; now on net HDMI_RX0_HOT: QRX001.1, RRX001.2
- net HDMIP_RX0_HPD renamed HDMIP_RX0_HOT
- net HDMI_RX0_HPA renamed HDMI_RX0_HOT
Other:
- note added: "This sheet is generated from ../external/templates/\nDO NOT MODIFY!!!\n4b96504"
- note removed: "This sheet is generated from ../external/templates/\nDO NOT MODIFY!!!\nedd182c"
Changed lines of the file:
@@
 VCC5V0_RX0
 Text Label 6150 4000 2    60   ~ 0
-HDMIP_RX0_HPD
+HDMIP_RX0_HOT
 Text Label 3525 5785 1    60   ~ 0
-HDMIP_RX0_HPD
+HDMIP_RX0_HOT
 Text Label 1500 6600 0    60   ~ 0
-HDMI_RX0_HPD
+HDMI_RX0_HOT
 Text Label 1500 7150 0    60   ~ 0
 GND
 Text Label 7560 6700 2    60   ~ 0
-HDMI_RX0_HPA
+HDMI_RX0_HOT
 Text Label 6750 1750 0    60   ~ 0
 GND
 Text HLabel 1500 6600 0    60   Input ~ 0
-HDMI_RX0_HPD
+HDMI_RX0_HOT
 Text Notes 615  11035 0    197  ~ 39
-This sheet is generated from ../external/templates/\nDO NOT MODIFY!!!\nedd182c
+This sheet is generated from ../external/templates/\nDO NOT MODIFY!!!\n4b96504
 Text Label 4820 6600 0    60   ~ 0
 HDMI_RX0_CEC

Commit message: Temp commit.
Changed lines of the file:
@@
 LIBS:contrib
 LIBS:valves
+LIBS:pmod
+LIBS:hdmi
+LIBS:ma78l00
 LIBS:pmod-conn_6x2
-LIBS:ma78l00
+LIBS:EEPROM
+LIBS:xc9140
+LIBS:reg710-dbv
+LIBS:ad8195
 LIBS:fdv301n
-LIBS:hdmi
-LIBS:ad8195
+LIBS:pmod-hdmi-rx-cache
 EELAYER 25 0
 EELAYER END
 $Descr A3 16535 11693
 encoding utf-8
-Sheet 1 1
+Sheet 2 2
 Title ""
 Date ""
@@
 U 1 1 57C077DA
 P 4750 3000
+AR Path="/57C077DA" Ref="JRX0"  Part="1"
+AR Path="/5802F547/57C077DA" Ref="JRX0"  Part="1"
 F 0 "JRX0" H 4600 4050 60  0000 C CNN
 F 1 "HDMI_IN" V 4900 3000 60  0000 C CNN
@@
 	7150 3650 6950 3650
 Wire Wire Line
-	6950 4900 6950 3650
-Wire Wire Line
-	5770 4900 6950 4900
+	6950 3650 6950 4900
+Wire Wire Line
+	6950 4900 5770 4900
 Wire Wire Line
 	7150 3750 7050 3750
 Wire Wire Line
-	7050 5000 7050 3750
-Wire Wire Line
-	5770 5000 7050 5000
+	7050 3750 7050 5000
+Wire Wire Line
+	7050 5000 5770 5000
 Wire Wire Line
 	6600 4900 6600 5150
