File: board/pmod-hdmi-tx.kicad_pcb (KiCad board)
At the start: 2 copper layers, 42 x 43.2 mm, 36 parts, among them P1 PMOD-Device-x2-Type-XHS-Alt, U31 XC9140, U32 REG710-DBV

Commit message: Fixing the via DRC violations.
Routing:
- net GND: track 454.9 -> 447.3 mm, vias 154 -> 149
- net (no net): track 6.65 -> 0.00 mm, vias 3 -> 0
- net VCC3V3: track 107.2 -> 102.1 mm
- net /HDMI TX/HDMIP_TX0_D2-: track 10.1 -> 10.6 mm
Other:
- net class Default: via_dia 0.6096 -> 0.6; via_drill 0.3048 -> 0.3
- net class HDMI_CAP2IC_DP0.0254/0.254 removed
- net class HDMI_IC2PORT_DP0.0254/0.381 removed
- net class HDMI_PMOD2CAP_DP0.0254/0.254 removed
- net class PWR: via_dia 0.6096 -> 0.6; via_drill 0.3048 -> 0.3
- rule via_min_drill: 0 -> 0.3
- rule via_min_size: 0.5 -> 0.6

Commit message: Clearance of 0.1269mm
Routing:
- net GND: track 447.3 -> 438.8 mm, vias 149 -> 147
- net (no net): track 0.00 -> 8.53 mm, vias 0 -> 2
Other:
- net class Default: clearance 0.127 -> 0.1269
- rule trace_clearance: 0.127 -> 0.1269
Changed lines of the file:
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@@
-(kicad_pcb (version 4) (host pcbnew 4.0.2-stable)
+(kicad_pcb (version 4) (host pcbnew 4.0.4+e1-6308~48~ubuntu14.04.1-stable)
   (general
     (links 102)
     (no_connects 1)
-    (area 48.707144 45.135715 236.364292 119.75)
+    (area 48.857144 45.285715 236.214292 120.05)
     (thickness 1.6)
     (drawings 131)
@@
     (last_trace_width 0.127)
     (user_trace_width 0.127)
-    (trace_clearance 0.127)
+    (trace_clearance 0.1269)
     (zone_clearance 0.2)
     (zone_45_only yes)
@@
   (net 47 "/HDMI TX/HDMIA_TX0_D2-")
   (net_class Default "This is the default net class."
-    (clearance 0.127)
+    (clearance 0.1269)
     (trace_width 0.127)
     (via_dia 0.6)
@@
   (gr_line (start 80.4 70.162) (end 80.4 113.342) (angle 90) (layer Edge.Cuts) (width 0.15))
   (gr_line (start 80.4 70.162) (end 122.4 70.162) (angle 90) (layer Edge.Cuts) (width 0.15))
+  (via (at 95.25 107.061) (size 0.6096) (drill 0.3048) (layers F.Cu B.Cu) (net 0))
+  (segment (start 90.17 107.061) (end 95.25 107.061) (width 0.25) (layer B.Cu) (net 0))
+  (segment (start 90.101 106.992) (end 90.17 107.061) (width 0.25) (layer F.Cu) (net 0))
+  (via (at 90.17 107.061) (size 0.6096) (drill 0.3048) (layers F.Cu B.Cu) (net 0))
+  (segment (start 88.6968 107.061) (end 92.0478 107.061) (width 0.25) (layer F.Cu) (net 0))
   (segment (start 107.315 109.22) (end 106.6546 108.5596) (width 0.25) (layer F.Cu) (net 1))
   (segment (start 106.6546 108.5596) (end 87.7224 108.5596) (width 0.25) (layer F.Cu) (net 1))
@@
   (via (at 95.25 92.71) (size 0.6096) (drill 0.3048) (layers F.Cu B.Cu) (net 2))
   (segment (start 99.822 92.71) (end 95.25 92.71) (width 0.25) (layer B.Cu) (net 2))
-  (via (at 95.25 107.061) (size 0.6096) (drill 0.3048) (layers F.Cu B.Cu) (net 2))
-  (segment (start 90.17 107.061) (end 95.25 107.061) (width 0.25) (layer B.Cu) (net 2))
-  (segment (start 90.101 106.992) (end 90.17 107.061) (width 0.25) (layer F.Cu) (net 2))
-  (via (at 90.17 107.061) (size 0.6096) (drill 0.3048) (layers F.Cu B.Cu) (net 2))
-  (segment (start 88.6968 107.061) (end 92.0478 107.061) (width 0.25) (layer F.Cu) (net 2))
   (segment (start 118.4148 102.3366) (end 119.6848 103.6066) (width 0.25) (layer B.Cu) (net 2))
   (segment (start 109.6518 102.2096) (end 114.0968 102.2096) (width 0.25) (layer B.Cu) (net 2))

Commit message: More fixes.
Parts:
- moved REF*** 2.01 mm to (99.5, 99.6)
Routing:
- net /HDMI_TX0_DDET: track 90.4 -> 90.9 mm
Other:
- net class Default: clearance 0.1269 -> 0.127
- rule trace_clearance: 0.1269 -> 0.127
- board text added: "$Id$"
- board text added: "CC-BY-SA 4.0"
- board text added: "https://mith.ro/gh /pmod-hdmi-tx /ptn3363"
- board text added: "tx0.2"
- board text removed: "647f4a6"
- board text removed: "pmod-hdmi-tx ptn3363"
- board text removed: "tx0.1"
Changed lines of the file:
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@@
   (general
     (links 102)
-    (no_connects 1)
+    (no_connects 0)
     (area 48.857144 45.285715 236.214292 120.05)
     (thickness 1.6)
-    (drawings 131)
-    (tracks 1778)
+    (drawings 132)
+    (tracks 1777)
     (zones 0)
     (modules 37)
@@
     (34 B.Paste user hide)
     (35 F.Paste user hide)
-    (36 B.SilkS user hide)
+    (36 B.SilkS user)
     (37 F.SilkS user hide)
     (38 B.Mask user hide)
@@
     (last_trace_width 0.127)
     (user_trace_width 0.127)
-    (trace_clearance 0.1269)
+    (trace_clearance 0.127)
     (zone_clearance 0.2)
     (zone_45_only yes)
@@
     (pad_to_mask_clearance 0.2)
     (aux_axis_origin 0 0)
-    (visible_elements 7FFFDE6D)
+    (visible_elements 7FFEDE6D)
     (pcbplotparams
       (layerselection 0x00030_80000001)
@@
   (net 47 "/HDMI TX/HDMIA_TX0_D2-")
   (net_class Default "This is the default net class."
-    (clearance 0.1269)
+    (clearance 0.127)
     (trace_width 0.127)
     (via_dia 0.6)
@@
     (tags "capacitor 0402")
     (attr smd)
-    (fp_text reference CTX013 (at -3.9536 0 90) (layer B.SilkS)
+    (fp_text reference CTX013 (at -1.887 -2.221 180) (layer B.SilkS)
       (effects (font (size 1 1) (thickness 0.15)) (justify mirror))
     )
@@
     (tags "Diode SOD523")
     (attr smd)
-    (fp_text reference DTX001 (at 0.0142 3.5306 180) (layer B.SilkS)
+    (fp_text reference DTX001 (at 0.5878 3.1734 90) (layer B.SilkS)
       (effects (font (size 1 1) (thickness 0.15)) (justify mirror))
     )
@@
     (tags "resistor 0402")
     (attr smd)
-    (fp_text reference RTX004 (at -4.1148 0.0762 90) (layer B.SilkS)
+    (fp_text reference RTX004 (at 3.82 0.064 90) (layer B.SilkS)
       (effects (font (size 1 1) (thickness 0.15)) (justify mirror))
     )
@@
     (tags "resistor 0402")
     (attr smd)
-    (fp_text reference RTX005 (at -4.1148 0.0508 90) (layer B.SilkS)
+    (fp_text reference RTX005 (at 3.82 0.017 90) (layer B.SilkS)
       (effects (font (size 1 1) (thickness 0.15)) (justify mirror))
     )
@@
   )
   (module Symbols:OSHW-Logo2_9.8x8mm_SilkScreen (layer F.Cu)
-    (at 100.203 101.473)
+    (at 99.475 99.6)
     (descr "Open Source Hardware Symbol")
     (tags "Logo Symbol OSHW")
@@
       (xy -0.017575 -3.712307) (xy 0 -3.712308) (xy 0.139878 -3.712224)) (layer F.SilkS) (width 0.01))
   )
+  (gr_text "CC-BY-SA 4.0" (at 99.475 104.325) (layer F.SilkS)
+    (effects (font (size 1 1) (thickness 0.25)))
+  )
   (gr_text C+ (at 81.7245 79.4385 180) (layer F.SilkS)
     (effects (font (size 1 1) (thickness 0.15)) (justify mirror))
@@
     (effects (font (size 1.5 1.5) (thickness 0.3)))
   )
-  (gr_text 647f4a6 (at 121.1072 109.2454) (layer B.SilkS)
+  (gr_text $Id$ (at 121.5 110.5) (layer B.SilkS)
     (effects (font (size 2.159 2.159) (thickness 0.53975)) (justify left mirror))
   )
-  (gr_text tx0.1 (at 121.0818 105.156) (layer B.SilkS)
+  (gr_text tx0.2 (at 121.5 106.5) (layer B.SilkS)
     (effects (font (size 2.159 2.159) (thickness 0.53975)) (justify left mirror))
   )
-  (gr_text "pmod-hdmi-tx\nptn3363" (at 121.2088 98.806) (layer B.SilkS)
+  (gr_text "https://mith.ro/gh\n/pmod-hdmi-tx\n/ptn3363" (at 121.5 98.5) (layer B.SilkS)
     (effects (font (size 2.159 2.159) (thickness 0.53975)) (justify left mirror))
   )
@@
   (segment (start 108.940596 80.962499) (end 111.061499 80.962499) (width 0.127) (layer B.Cu) (net 19))
   (segment (start 111.061499 80.962499) (end 111.252 81.153) (width 0.127) (layer B.Cu) (net 19))
-  (via (at 111.2774 81.153) (size 0.6096) (drill 0.3048) (layers F.Cu B.Cu) (net 19))
+  (via (at 111.25 81.153) (size 0.6096) (drill 0.3048) (layers F.Cu B.Cu) (net 19))
   (segment (start 111.429 81.33) (end 111.252 81.153) (width 0.127) (layer F.Cu) (net 19))
   (segment (start 113.136 81.33) (end 111.429 81.33) (width 0.127) (layer F.Cu) (net 19))
@@
   (segment (start 100.264 76.374875) (end 100.264 77.47) (width 0.127) (layer B.Cu) (net 32))
   (segment (start 100.264 79.437) (end 100.264 79.914) (width 0.127) (layer B.Cu) (net 32))
-  (segment (start 87.5792 100.723575) (end 86.195025 100.723575) (width 0.127) (layer B.Cu) (net 33))
-  (segment (start 100.764 79.914) (end 100.764 79.1232) (width 0.127) (layer B.Cu) (net 33))
-  (segment (start 85.797499 105.404501) (end 86.75 104.452) (width 0.127) (layer B.Cu) (net 33))
-  (segment (start 100.764 79.1232) (end 100.6602 79.0194) (width 0.127) (layer B.Cu) (net 33))
-  (segment (start 83.185 103.8352) (end 83.185 105.0544) (width 0.127) (layer B.Cu) (net 33))
-  (segment (start 100.6602 79.0194) (end 100.6602 78.539) (width 0.127) (layer B.Cu) (net 33))
-  (segment (start 89.438763 98.864012) (end 87.5792 100.723575) (width 0.127) (layer B.Cu) (net 33))
-  (segment (start 100.6602 78.539) (end 100.764 78.4352) (width 0.127) (layer B.Cu) (net 33))
-  (segment (start 100.764 78.4352) (end 100.764 75.8023) (width 0.127) (layer B.Cu) (net 33))
-  (segment (start 85.6234 102.108) (end 84.6074 103.124) (width 0.127) (layer B.Cu) (net 33))
-  (segment (start 83.6676 105.537) (end 85.6488 105.537) (width 0.127) (layer B.Cu) (net 33))
-  (segment (start 100.764 75.8023) (end 104.30923 72.25707) (width 0.127) (layer B.Cu) (net 33))
-  (segment (start 104.30923 72.25707) (end 116.87397 72.25707) (width 0.127) (layer B.Cu) (net 33))
-  (segment (start 116.87397 72.25707) (end 118.163329 73.546429) (width 0.127) (layer B.Cu) (net 33))
-  (segment (start 89.455213 98.864012) (end 89.438763 98.864012) (width 0.127) (layer B.Cu) (net 33))
-  (segment (start 118.163329 73.546429) (end 118.163329 94.452796) (width 0.127) (layer B.Cu) (net 33))
-  (segment (start 118.163329 94.452796) (end 116.12147 96.494655) (width 0.127) (layer B.Cu) (net 33))
-  (segment (start 86.195025 100.723575) (end 85.6234 101.2952) (width 0.127) (layer B.Cu) (net 33))
-  (segment (start 116.12147 96.494655) (end 91.82457 96.494655) (width 0.127) (layer B.Cu) (net 33))
-  (segment (start 91.82457 96.494655) (end 89.455213 98.864012) (width 0.127) (layer B.Cu) (net 33))
-  (segment (start 85.6234 101.2952) (end 85.6234 102.108) (width 0.127) (layer B.Cu) (net 33))
-  (segment (start 83.8962 103.124) (end 83.185 103.8352) (width 0.127) (layer B.Cu) (net 33))
-  (segment (start 84.6074 103.124) (end 83.8962 103.124) (width 0.127) (layer B.Cu) (net 33))
-  (segment (start 83.185 105.0544) (end 83.6676 105.537) (width 0.127) (layer B.Cu) (net 33))
-  (segment (start 85.6488 105.537) (end 85.781299 105.404501) (width 0.127) (layer B.Cu) (net 33))
-  (segment (start 85.781299 105.404501) (end 85.797499 105.404501) (width 0.127) (layer B.Cu) (net 33))
-  (segment (start 100.203 77.724) (end 100.51 77.724) (width 0.127) (layer F.Cu) (net 33))
-  (segment (start 100.51 77.724) (end 100.764 77.978) (width 0.127) (layer F.Cu) (net 33))
-  (via (at 100.8126 77.724) (size 0.6096) (drill 0.3048) (layers F.Cu B.Cu) (net 33))
+  (segment (start 100.9 77.31893) (end 100.9 77.749982) (width 0.127) (layer B.Cu) (net 33))
+  (segment (start 116.87397 72.25707) (end 104.30923 72.25707) (width 0.127) (layer B.Cu) (net 33))
+  (segment (start 86.195025 100.723575) (end 87.5792 100.723575) (width 0.127) (layer B.Cu) (net 33))
+  (segment (start 118.163329 94.452796) (end 118.163329 73.546429) (width 0.127) (layer B.Cu) (net 33))
+  (segment (start 89.455213 98.864012) (end 91.82457 96.494655) (width 0.127) (layer B.Cu) (net 33))
+  (segment (start 89.438763 98.864012) (end 89.455213 98.864012) (width 0.127) (layer B.Cu) (net 33))
+  (segment (start 116.12147 96.494655) (end 118.163329 94.452796) (width 0.127) (layer B.Cu) (net 33))
+  (segment (start 104.30923 72.25707) (end 100.9 75.6663) (width 0.127) (layer B.Cu) (net 33))
+  (segment (start 87.5792 100.723575) (end 89.438763 98.864012) (width 0.127) (layer B.Cu) (net 33))
+  (segment (start 85.6234 101.2952) (end 86.195025 100.723575) (width 0.127) (layer B.Cu) (net 33))
+  (segment (start 85.6234 102.108) (end 85.6234 101.2952) (width 0.127) (layer B.Cu) (net 33))
+  (segment (start 84.6074 103.124) (end 85.6234 102.108) (width 0.127) (layer B.Cu) (net 33))
+  (segment (start 91.82457 96.494655) (end 116.12147 96.494655) (width 0.127) (layer B.Cu) (net 33))
+  (segment (start 83.8962 103.124) (end 84.6074 103.124) (width 0.127) (layer B.Cu) (net 33))
+  (segment (start 83.185 105.0544) (end 83.185 103.8352) (width 0.127) (layer B.Cu) (net 33))
+  (segment (start 100.9 75.6663) (end 100.9 77.31893) (width 0.127) (layer B.Cu) (net 33))
+  (segment (start 118.163329 73.546429) (end 116.87397 72.25707) (width 0.127) (layer B.Cu) (net 33))
+  (segment (start 83.185 103.8352) (end 83.8962 103.124) (width 0.127) (layer B.Cu) (net 33))
+  (segment (start 85.665 105.537) (end 83.6676 105.537) (width 0.127) (layer B.Cu) (net 33))
+  (segment (start 86.75 104.452) (end 85.665 105.537) (width 0.127) (layer B.Cu) (net 33))
+  (segment (start 100.764 77.885982) (end 100.9 77.749982) (width 0.127) (layer B.Cu) (net 33))
+  (segment (start 100.764 79.914) (end 100.764 77.885982) (width 0.127) (layer B.Cu) (net 33))
+  (segment (start 83.6676 105.537) (end 83.185 105.0544) (width 0.127) (layer B.Cu) (net 33))
+  (segment (start 100.874018 77.724) (end 100.9 77.749982) (width 0.127) (layer F.Cu) (net 33))
+  (segment (start 100.203 77.724) (end 100.874018 77.724) (width 0.127) (layer F.Cu) (net 33))
+  (via (at 100.9 77.749982) (size 0.6096) (drill 0.3048) (layers F.Cu B.Cu) (net 33))
+  (segment (start 100.203 77.724) (end 100.76 77.724) (width 0.127) (layer F.Cu) (net 33))
+  (segment (start 100.76 77.724) (end 100.764 77.728) (width 0.127) (layer F.Cu) (net 33))
   (segment (start 100.764 79.437) (end 100.764 79.914) (width 0.127) (layer B.Cu) (net 33))
   (segment (start 94.615 100.7618) (end 100.711 94.6658) (width 0.127) (layer F.Cu) (net 34))

Commit message: A bunch of cleanup, see detailed comment below.
* Reorganized value labels for a better manual placement plan.
* Replaced manually created dimensions using KiCad dimension object.
* Removed dimensions that were not anchored to anything obviously
  useful. I assume they are cutandpasta remains.
* Removed floating items on the Cmts.User layer.
* Fab notes merged into a single object. There is no need to write the
  text in multiple separate strings and arrange them manually, even if
  it is autogenerated.
Other:
- board text added: "NOTES: (UNLESS OTHERWISE SPECIFIED) 1. MATERIAL: FR408 1.6 mm THK, 4 LAYERS, EQUALLY SPACED, 1 OZ CU ALL LAYERS, WHEN FINISHED. 2. PLATED HOLES TO HAVE 1/2 OZ CU MIN. 3. PURPLE SOLDERMASK OVER BARE CU, BOTH SIDES. 4. ENIG (ELECTROLESS NICKEL IMMERSION GOLD) 5. PERMANENTLY MARK DATE CODE AND MANUFACTURING SYMBOL ON BOTTOM."
- board text removed: "1 OZ CU ALL LAYERS, WHEN FINISHED."
- board text removed: "1. MATERIAL: FR408 1.6 mm THK, 4 LAYERS, EQUALLY SPACED,"
- board text removed: "101.4"
- board text removed: "104.5"
- board text removed: "113.342"
- board text removed: "122.4"
- board text removed: "2. PLATED HOLES TO HAVE 1/2 OZ CU MIN."
- board text removed: "2.842"
- board text removed: "21.0"
- board text removed: "3. PURPLE SOLDERMASK OVER BARE CU, BOTH SIDES."
- board text removed: "31.496"
- board text removed: "4. ENIG (ELECTROLESS NICKEL IMMERSION GOLD)"
- board text removed: "42.0"
- board text removed: "43.18"
- board text removed: "5. PERMANENTLY MARK DATE CODE AND"
- board text removed: "70.162"
- board text removed: "73.004"
- board text removed: "76.0"
- board text removed: "80.4"
- board text removed: "91.0"
- board text removed: "MANUFACTURING SYMBOL ON BOTTOM."
- board text removed: "NOTES: (UNLESS OTHERWISE SPECIFIED)"
